File: esp_hat.sch (KiCad schematic (older format))
At the start: 36 parts, among them IC1 AT24CS32-STUM, J1 U.FL, P1 CONN_02X20, P2 CONN_01X03, P3 CONN_01X06, U1 ESP8266EX, U2 AP1117D33, Y1 26MHz

Commit message: Mostly done
Parts:
- Y1: footprint Crystals:Crystal_SMD_0603_4Pads -> Crystals:crystal_FA238-TSX3225
Changed lines of the file:
@@
 F 0 "Y1" H 2150 5200 50  0000 C CNN
 F 1 "26MHz" H 2150 4900 50  0000 C CNN
-F 2 "Crystals:Crystal_SMD_0603_4Pads" H 2150 5050 50  0001 C CNN
+F 2 "Crystals:crystal_FA238-TSX3225" H 2150 5050 50  0001 C CNN
 F 3 "" H 2150 5050 50  0000 C CNN
 	1    2150 5050
