File: esp_hat.sch (KiCad schematic (older format))
At the start: 36 parts, among them IC1 AT24CS32-STUM, J1 U.FL, P1 CONN_02X20, P2 CONN_01X03, P3 CONN_01X06, U1 ESP8266EX, U2 AP1117D33, Y1 26MHz

Commit message: commit v0.2 changes, remove v0.1 fab files
Parts:
- removed C4: 10uF, mcuos:0603(1608m)-CHIP-CAP, symbol C
- removed IC1: AT24CS32-STUM, TO_SOT_Packages_SMD:SOT-23-5, symbol AT24CS32-STUM
- removed JP1: Jumper_NO_Small, Connect:GS2, symbol Jumper_NO_Small
- removed P2: CONN_01X03, Pin_Headers:Pin_Header_Straight_1x03, symbol CONN_01X03
- removed P3: CONN_01X06, Pin_Headers:Pin_Header_Straight_1x06, symbol CONN_01X06
- removed R13: 1K, mcuos:0603(1608m)-CHIP-RESISTOR, symbol R
- removed R14, R15: 3.9K, mcuos:0603(1608m)-CHIP-RESISTOR, symbol R
- added W1: RXD, Measurement_Points:Measurement_Point_Round-SMD-Pad_Small, symbol TEST_1P
- added W2: TXD, Measurement_Points:Measurement_Point_Round-SMD-Pad_Small, symbol TEST_1P
- added W3, W4, W5, W6: MOUNT, esp_hat:NPTH_Hole_2_75mm, symbol TEST_1P
- ANT1: footprint SH_Antennas:TI_DN007_2.4GHz -> esp_hat:TI_DN007_2.4GHz
- C5: value 1uF -> 0.1uF
- R1: renamed from R11; footprint mcuos:0603(1608m) -> mcuos:0603(1608m)-CHIP-RESISTOR
- R3: renamed from R1; footprint mcuos:0603(1608m) -> Connect:GS2
- R4: renamed from R2; footprint mcuos:0603(1608m) -> Connect:GS2
- R5: renamed from R3; footprint mcuos:0603(1608m) -> Connect:GS2
- U2: footprint TO_SOT_Packages_SMD:SOT-223 -> esp_hat:SOT-223-REG_VOUTSLUG
- renumbered C3 to C2, C2 to C3, C6 to C4, C7 to C6, C8 to C7, R8 to R10, R9 to R11, R10 to R12, R12 to R2, R4 to R6, R5 to R7, R6 to R8, R7 to R9
Connections:
- net labels removed: ID_SC, ID_SD, PI_UART0_RXD, PI_UART0_TXD
- wire segments 126 -> 96
- no-connect marks 32 -> 33
Other:
- note removed: "Short for HAT config\nSEEP write enable"
- moved on the sheet: C1, C2, C4, Y1

Commit message: Add GPIO5/GPIO6 select pad, fix no-connects, remove paste on option pads
Parts:
- added P2: CONN_01X03, esp_hat:GS3, symbol CONN_01X03
Connections:
- net labels added: GPIO6
- wire segments 96 -> 102
- no-connect marks 33 -> 32
Changed lines of the file:
@@
 LIBS:valves
 LIBS:esp_hat
+LIBS:esp_hat-cache
 EELAYER 25 0
 EELAYER END
@@
 Sheet 1 1
 Title "ESP HAT"
-Date "2015-12-31"
+Date "2016-01-01"
 Rev "v0.2"
 Comp "Andrew Litt"
@@
 Text GLabel 8550 3750 0    39   BiDi ~ 0
 GPIO5
-Text GLabel 2350 4050 0    39   Input ~ 0
+Text GLabel 1600 4400 2    39   Input ~ 0
 GPIO5
 $Comp
@@
 NoConn ~ 9200 3450
 NoConn ~ 9200 3550
-NoConn ~ 8700 3850
 NoConn ~ 8700 3950
 NoConn ~ 8700 4050
@@
 	6350 1600 6350 1750
 Connection ~ 6350 1600
+Text GLabel 8550 3850 0    39   BiDi ~ 0
+GPIO6
+Wire Wire Line
+	8550 3850 8700 3850
+$Comp
+L CONN_01X03 P2
+U 1 1 5686E4DE
+P 1200 4300
+F 0 "P2" H 1200 4500 50  0000 C CNN
+F 1 "CONN_01X03" V 1300 4300 50  0000 C CNN
+F 2 "esp_hat:GS3" H 1200 4300 50  0001 C CNN
+F 3 "" H 1200 4300 50  0000 C CNN
+	1    1200 4300
+	-1   0    0    1
+$EndComp
+Text GLabel 1600 4200 2    39   Input ~ 0
+GPIO6
+Wire Wire Line
+	2350 4050 2350 4300
+Wire Wire Line
+	2350 4300 1400 4300
+Wire Wire Line
+	1400 4200 1600 4200
+Wire Wire Line
+	1400 4400 1600 4400
+Wire Wire Line
+	1450 4300 1450 4400
+Connection ~ 1450 4400
+Connection ~ 1450 4300
 $EndSCHEMATC

Commit message: Add part# parameters, clean up refs, set attributes for proper mfg
Parts:
- removed P2: CONN_01X03, esp_hat:GS3, symbol CONN_01X03
- removed R10, R11, R12: 200, mcuos:0603(1608m)-CHIP-RESISTOR, symbol R
- removed R3: DNP, Connect:GS2, symbol R
- added JP1: CHIP_EN, esp_hat:GS3, symbol JUMPER3
- added JP2: MTDO, esp_hat:GS2, symbol JUMPER
- added JP3: GPIO2, esp_hat:GS2, symbol JUMPER
- added JP4: GPIO0, esp_hat:GS2, symbol JUMPER
- added R6: 200, mcuos:0603(1608m)-CHIP-RESISTOR, symbol R
- C1, C2: 2nd Distrib Link (none) -> NA; 2nd Distrib PN (none) -> NA; Digikey Link (none) -> https://www.digikey.com/product-detail/en/C0603C100J5GACTU/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; Digikey PN (none) -> 399-1049-1-ND; MFG Name (none) -> Kemet; MFG Part Num (none) -> C0603C100J5GACTU
- C3: 1st Distrib Link (none) -> https://www.digikey.com/product-detail/en/251R14S5R6CV4T/71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; 1st Distrib PN (none) -> 712-1360-1-ND; 2nd Distrib Link (none) -> NA; 2nd Distrib PN (none) -> NA; MFG Name (none) -> Johanson Technology Inc.; MFG Part Num (none) -> 251R14S5R6CV4T
- C4, C5: 2nd Distrib Link (none) -> NA; 2nd Distrib PN (none) -> NA; Digikey Link (none) -> https://www.digikey.com/product-detail/en/GRM188R71C104KA01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; Digikey PN (none) -> 490-1532-1-ND; MFG Name (none) -> Murata Electronics North America; MFG Part Num (none) -> GRM188R71C104KA01D
- C6, C7: 2nd Distrib Link (none) -> NA; 2nd Distrib PN (none) -> NA; Digikey Link (none) -> https://www.digikey.com/product-detail/en/GRM188R60J106ME47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; Digikey PN (none) -> 490-6405-1-ND; MFG Name (none) -> Murata Electronics North America; MFG Part Num (none) -> GRM188R60J106ME47J
- FB1: footprint mcuos:0603(1608m) -> mcuos:0603(1608m)-CHIP-CAP; 2nd Distrib Link (none) -> NA; 2nd Distrib PN (none) -> NA; Digikey Link (none) -> https://www.digikey.com/product-detail/en/BLM18AG601SN1D/49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; Digikey PN (none) -> 490-1014-1-ND; MFG Name (none) -> Murata Electronics North America; MFG Part Num (none) -> BLM18AG601SN1D
- J1: value U.FL -> DNP; 2nd Distrib Link (none) -> NA; 2nd Distrib PN (none) -> NA; Digikey Link (none) -> https://www.digikey.com/product-detail/en/U.FL-R-SMT(01)/H9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; Digikey PN (none) -> H9161-ND; MFG Name (none) -> Hirose Electric Co Ltd; MFG Part Num (none) -> U.FL-R-SMT(01)
- L1, L2: footprint mcuos:0603(1608m) -> mcuos:0603(1608m)-CHIP-CAP
- P1: 2nd Distrib Link (none) -> NA; 2nd Distrib PN (none) -> NA; Digikey Link (none) -> http://www.digikey.com/product-search/en?pv88=23&FV=fff4001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; Digikey PN (none) -> 1528-1385-ND; MFG Name (none) -> Adafruit Industries; MFG Part Num (none) -> 2223
- R1, R2: 2nd Distrib Link (none) -> NA; 2nd Distrib PN (none) -> NA; Digikey Link (none) -> https://www.digikey.com/product-detail/en/ERJ-3GEY0R00V/P0.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; Digikey PN (none) -> P0.0GCT-ND; MFG Name (none) -> Panasonic Electronic Components; MFG Part Num (none) -> ERJ-3GEY0R00V
- R3: renamed from R6; value 12.0K -> 12.0K 1%; 2nd Distrib Link (none) -> NA; 2nd Distrib PN (none) -> NA; Digikey Link (none) -> NA; Digikey PN (none) -> P12.0HCT-ND; MFG Name (none) -> Panasonic Electronic Components; MFG Part Num (none) -> ERJ-3EKF12R0V
- R4, R5: value DNP -> 200; footprint Connect:GS2 -> mcuos:0603(1608m)-CHIP-RESISTOR; 2nd Distrib Link (none) -> NA; 2nd Distrib PN (none) -> NA; Digikey Link (none) -> https://www.digikey.com/product-detail/en/ERJ-3EKF2000V/P20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; Digikey PN (none) -> P200HCT-ND; MFG Name (none) -> Panasonic Electronic Components; MFG Part Num (none) -> ERJ-3EKF2000V
- R7, R8, R9: 2nd Distrib Link (none) -> NA; 2nd Distrib PN (none) -> NA; Digikey Link (none) -> https://www.digikey.com/product-detail/en/ERJ-3EKF2000V/P20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; Digikey PN (none) -> P200HCT-ND; MFG Name (none) -> Panasonic Electronic Components; MFG Part Num (none) -> ERJ-3EKF2000V
- U1: 1st Distrib Link (none) -> NA; 1st Distrib PN (none) -> NA; 2nd Distrib Link (none) -> NA; 2nd Distrib PN (none) -> NA; MFG Name (none) -> Espressif; MFG Part Num (none) -> ESP8266EX
- U2: 2nd Distrib Link (none) -> NA; 2nd Distrib PN (none) -> NA; Digikey Link (none) -> https://www.digikey.com/product-detail/en/AP1117E33G-13/AP1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; Digikey PN (none) -> AP1117E33GDICT-ND; MFG Name (none) -> Diodes Incorporated; MFG Part Num (none) -> AP1117E33G-13
- W1, W2: footprint Measurement_Points:Measurement_Point_Round-SMD-Pad_Small -> esp_hat:Measurement_Point_Round-SMD-Pad_Small; 2nd Distrib Link (none) -> NA; 2nd Distrib PN (none) -> NA; Digikey Link (none) -> NA; Digikey PN (none) -> NA; MFG Name (none) -> NA; MFG Part Num (none) -> NA
- Y1: value 26MHz -> 26MHz 10ppm; 2nd Distrib Link (none) -> NA; 2nd Distrib PN (none) -> NA; Digikey Link (none) -> https://www.digikey.com/product-detail/en/NX3225SA-26.000M-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; Digikey PN (none) -> 44-1269-1-ND; MFG Name (none) -> NDK; MFG Part Num (none) -> NX3225SA-26.000M-STD-CSQ-1
Other:
- moved on the sheet: R3
